File: pt2lcd-breakoutboard.kicad_pcb (KiCad board)
At the start: 2 copper layers, 74 x 142 mm, 19 parts, among them J1 PWRCONN, J3 PROTOCONN, SW1 BACK, SW2 UP, SW3 MID, SW4 DOWN, U1 BM20B0.6-24DS-0.4V53, U2 LT3009

Commit message: changed trace spacing
Routing:
- net GND: vias 9 -> 13
Changed lines of the file:
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@@
 			(plot_on_all_layers_selection 0x0000000_00000000)
 			(disableapertmacros no)
-			(usegerberextensions no)
-			(usegerberattributes yes)
-			(usegerberadvancedattributes yes)
-			(creategerberjobfile yes)
+			(usegerberextensions yes)
+			(usegerberattributes no)
+			(usegerberadvancedattributes no)
+			(creategerberjobfile no)
 			(dashed_line_dash_ratio 12.000000)
 			(dashed_line_gap_ratio 3.000000)
@@
 			(plotinvisibletext no)
 			(sketchpadsonfab no)
-			(subtractmaskfromsilk no)
+			(subtractmaskfromsilk yes)
 			(outputformat 1)
 			(mirror no)
-			(drillshape 1)
+			(drillshape 0)
 			(scaleselection 1)
-			(outputdirectory "")
+			(outputdirectory "Gerber/")
 		)
 	)
@@
 		)
 		(height -50.11)
-		(gr_text "12.8000 mm"
+		(gr_text "12,8000 mm"
 			(at 125.08 70.96 0)
 			(layer "Dwgs.User")
@@
 		)
 		(height -2.82)
-		(gr_text "50.0800 mm"
+		(gr_text "50,0800 mm"
 			(at 114.06 97.83 90)
 			(layer "Dwgs.User")
@@
 	)
 	(via
+		(at 134.5 119.5)
+		(size 0.6)
+		(drill 0.3)
+		(layers "F.Cu" "B.Cu")
+		(free yes)
+		(net 1)
+	)
+	(via
 		(at 138.92 108.11)
 		(size 0.6)
@@
 	)
 	(via
+		(at 134 111)
+		(size 0.6)
+		(drill 0.3)
+		(layers "F.Cu" "B.Cu")
+		(free yes)
+		(net 1)
+	)
+	(via
 		(at 154 100)
 		(size 0.6)
@@
 		(net 1)
 	)
+	(via
+		(at 144 111)
+		(size 0.6)
+		(drill 0.3)
+		(layers "F.Cu" "B.Cu")
+		(free yes)
+		(net 1)
+	)
+	(via
+		(at 144 108)
+		(size 0.6)
+		(drill 0.3)
+		(layers "F.Cu" "B.Cu")
+		(free yes)
+		(net 1)
+	)
 	(segment
 		(start 139.420197 113.825)
@@
 	)
 	(segment
-		(start 136.022199 135.057199)
-		(end 136.640957 135.057199)
-		(width 0.15)
-		(layer "F.Cu")
-		(net 7)
-	)
-	(segment
-		(start 123.662399 122.697399)
-		(end 136.022199 135.057199)
+		(start 119.830076 122.697399)
+		(end 123.662399 122.697399)
 		(width 0.15)
 		(layer "F.Cu")
@@
 	)
 	(segment
-		(start 119.830076 122.697399)
-		(end 123.662399 122.697399)
+		(start 123.677798 122.682)
+		(end 125.222 122.682)
 		(width 0.15)
 		(layer "F.Cu")
@@
 	)
 	(segment
-		(start 137.299966 135.716208)
-		(end 137.299966 136.182199)
+		(start 138.714966 136.174966)
+		(end 138.714966 136.182199)
 		(width 0.15)
 		(layer "F.Cu")
@@
 	)
 	(segment
-		(start 136.640957 135.057199)
-		(end 137.299966 135.716208)
+		(start 123.662399 122.697399)
+		(end 123.677798 122.682)
 		(width 0.15)
 		(layer "F.Cu")
@@
 	)
 	(segment
-		(start 137.299966 136.182199)
-		(end 138.714966 136.182199)
+		(start 125.222 122.682)
+		(end 138.714966 136.174966)
 		(width 0.15)
 		(layer "F.Cu")
@@
 	)
 	(segment
-		(start 119.830076 120.697397)
-		(end 128.012397 120.697397)
+		(start 147.058767 131.826)
+		(end 151.414966 136.182199)
 		(width 0.15)
 		(layer "F.Cu")
@@
 	)
 	(segment
-		(start 148.539966 133.307199)
-		(end 151.414966 136.182199)
+		(start 129.841397 120.697397)
+		(end 140.97 131.826)
 		(width 0.15)
 		(layer "F.Cu")
@@
 	)
 	(segment
-		(start 140.622199 133.307199)
-		(end 148.539966 133.307199)
+		(start 140.97 131.826)
+		(end 147.058767 131.826)
 		(width 0.15)
 		(layer "F.Cu")
@@
 	)
 	(segment
-		(start 128.012397 120.697397)
-		(end 140.622199 133.307199)
+		(start 119.830076 120.697397)
+		(end 129.841397 120.697397)
 		(width 0.15)
 		(layer "F.Cu")
@@
 	)
 	(segment
-		(start 137.862199 134.357199)
-		(end 141.969966 134.357199)
+		(start 126.98345 121.897398)
+		(end 139.249292 134.16324)
 		(width 0.15)
 		(layer "F.Cu")
@@
 	)
 	(segment
-		(start 141.969966 134.357199)
-		(end 143.794966 136.182199)
+		(start 119.830076 121.897398)
+		(end 126.98345 121.897398)
 		(width 0.15)
 		(layer "F.Cu")
@@
 	)
 	(segment
-		(start 125.402398 121.897398)
-		(end 137.862199 134.357199)
+		(start 139.249292 134.16324)
+		(end 141.776007 134.16324)
 		(width 0.15)
 		(layer "F.Cu")
@@
 	)
 	(segment
-		(start 119.830076 121.897398)
-		(end 125.402398 121.897398)
+		(start 141.776007 134.16324)
+		(end 143.794966 136.182199)
 		(width 0.15)
 		(layer "F.Cu")
@@
 	)
 	(segment
-		(start 124.532399 122.297399)
-		(end 136.942199 134.707199)
+		(start 139.779966 134.707199)
+		(end 141.254966 136.182199)
 		(width 0.15)
 		(layer "F.Cu")
@@
 	)
 	(segment
-		(start 139.779966 134.707199)
-		(end 141.254966 136.182199)
+		(start 126.288906 122.297399)
+		(end 138.698706 134.707199)
 		(width 0.15)
 		(layer "F.Cu")
@@
 	)
 	(segment
-		(start 119.830076 122.297399)
-		(end 124.532399 122.297399)
+		(start 138.698706 134.707199)
+		(end 139.779966 134.707199)
 		(width 0.15)
 		(layer "F.Cu")
@@
 	)
 	(segment
-		(start 136.942199 134.707199)
-		(end 139.779966 134.707199)
+		(start 119.830076 122.297399)
+		(end 126.288906 122.297399)
 		(width 0.15)
 		(layer "F.Cu")
@@
 	)
 	(segment
-		(start 119.830076 121.097399)
-		(end 127.142399 121.097399)
+		(start 140.328844 132.708844)
+		(end 145.401611 132.708844)
 		(width 0.15)
 		(layer "F.Cu")
@@
 	)
 	(segment
-		(start 139.702199 133.657199)
-		(end 146.349966 133.657199)
+		(start 119.830076 121.097399)
+		(end 128.717399 121.097399)
 		(width 0.15)
 		(layer "F.Cu")
@@
 	)
 	(segment
-		(start 146.349966 133.657199)
+		(start 145.401611 132.708844)
 		(end 148.874966 136.182199)
 		(width 0.15)
@@
 	)
 	(segment
-		(start 127.142399 121.097399)
-		(end 139.702199 133.657199)
+		(start 128.717399 121.097399)
+		(end 140.328844 132.708844)
 		(width 0.15)
 		(layer "F.Cu")
@@
 	)
 	(segment
-		(start 126.272398 121.497398)
-		(end 138.782199 134.007199)
+		(start 119.830076 121.497398)
+		(end 127.847398 121.497398)
 		(width 0.15)
 		(layer "F.Cu")
@@
 	)
 	(segment
-		(start 138.782199 134.007199)
-		(end 144.159966 134.007199)
+		(start 143.756767 133.604)
+		(end 146.334966 136.182199)
 		(width 0.15)
 		(layer "F.Cu")
@@
 	)
 	(segment
-		(start 144.159966 134.007199)
-		(end 146.334966 136.182199)
+		(start 139.954 133.604)
+		(end 143.756767 133.604)
 		(width 0.15)
 		(layer "F.Cu")
@@
 	)
 	(segment
-		(start 119.830076 121.497398)
-		(end 126.272398 121.497398)
+		(start 127.847398 121.497398)
+		(end 139.954 133.604)
 		(width 0.15)
 		(layer "F.Cu")
